Commit message: latest

File: model/BlueRov2.urdf.xacro (robot description, xacro)
@@ -81,5 +81,5 @@
       <origin xyz="0 0 0" rpy="0 0 0"/>
       <geometry>
-        <mesh filename="package://bluerov_ros_playground/model/BlueRov2.dae"/>
+        <mesh filename="package://bluerov_ros/model/BlueRov2.dae"/>
       </geometry>
     </visual>
